Commit message: 1223_0842_更换了urdf

File: general_motion_tracker_whole_body_teleoperation/general_motion_tracker_whole_body_teleoperation/assets/Q1/urdf/Q1_wo_hand_rl.urdf (robot description, URDF)
Before this commit: robot Q1_wo_hand, 30 links, 29 joints
Links:
- link L_ankle_pitch_link: mass 0.00495302360887897 -> 0.046
- link L_ankle_roll_link: mass 0.700527444039911 -> 0.7
- link L_elbow_link: mass 0.25017827413194 -> 0.25
- link L_forearm_yaw_link: mass 1.04944082700571 -> 1.05
- link L_hip_pitch_link: mass 2.04935184270293 -> 2.05
- link L_hip_roll_link: mass 1.25324354201009 -> 1.25
- link L_hip_yaw_link: mass 3.64631909766459 -> 3.65
- link L_knee_link: mass 5.84550624070991 -> 5.85
- link L_shoulder_pitch_link: mass 1.50011760905892 -> 1.35
- link L_shoulder_roll_link: mass 0.548488874404492 -> 0.55
- link L_shoulder_yaw_link: mass 1.95077707562053 -> 1.95
- link L_wrist_pitch_link: mass 0.150455726882542 -> 0.16
- link L_wrist_roll_link: mass 0.24994172305006 -> 0.25
- link R_ankle_pitch_link: mass 0.00495302360887897 -> 0.046
- link R_ankle_roll_link: mass 0.700527402465685 -> 0.7
- link R_elbow_link: mass 0.250208538636712 -> 0.25
- link R_forearm_yaw_link: mass 1.04948017603507 -> 1.05
- link R_hip_pitch_link: mass 2.04935276321242 -> 2.05
- link R_hip_roll_link: mass 1.25324353787124 -> 1.25
- link R_hip_yaw_link: mass 3.64637969927244 -> 3.65
- link R_knee_link: mass 5.84551012436571 -> 5.85
- link R_shoulder_pitch_link: mass 1.50011657804918 -> 1.35
- link R_shoulder_roll_link: mass 0.548544608828653 -> 0.55
- link R_shoulder_yaw_link: mass 1.95078429643153 -> 1.95
- link R_wrist_pitch_link: mass 0.150463482385983 -> 0.16
- link R_wrist_roll_link: mass 0.249941692839846 -> 0.25
- link head_pitch_link: mass 0.8024 -> 0.72904
- link head_yaw_link: mass 0.801875605020622 -> 0.8
- link pelvis_link: mass 4.85375453300402 -> 4.85
- link torso_link: mass 15.889 -> 19.078
Joints:
- joint L_ankle_pitch_joint: origin xyz=0 0 -0.451 rpy=0 0 0 -> xyz=0 -1.39E-05 -0.45087 rpy=0 0 0
- joint L_forearm_yaw_joint: origin xyz=0 0 -0.231 rpy=0 0 0 -> xyz=0 0 -0.209 rpy=0 0 0
- joint L_hip_roll_joint: origin xyz=0 0.115 -0.05874 rpy=0 0 0 -> xyz=-9.9986E-05 0.115 -0.059738 rpy=0 0 0
- joint L_knee_joint: origin xyz=0 0 -0.285 rpy=0 0 0 -> xyz=0 0 -0.28496 rpy=0 0 0
- joint L_shoulder_pitch_joint: origin xyz=0 0.2222 0.37445 rpy=0.2618 0 0 -> xyz=-0.00015827 0.22119 0.38344 rpy=0.2618 0 0
- joint L_shoulder_yaw_joint: origin xyz=0 -0.043643 -0.25143 rpy=-0.2618 0 0 -> xyz=0 -0.043208 -0.25042 rpy=-0.2618 0 0
- joint R_ankle_pitch_joint: origin xyz=0 0 -0.451 rpy=0 0 0 -> xyz=0 1.39E-05 -0.45087 rpy=0 0 0
- joint R_forearm_yaw_joint: origin xyz=0 0 -0.231 rpy=0 0 0 -> xyz=0 0 -0.209 rpy=0 0 0
- joint R_hip_roll_joint: origin xyz=0 -0.115 -0.05874 rpy=0 0 0 -> xyz=-9.9986E-05 -0.115 -0.059738 rpy=0 0 0
- joint R_knee_joint: origin xyz=0 0 -0.285 rpy=0 0 0 -> xyz=0 0 -0.28496 rpy=0 0 0
- joint R_shoulder_pitch_joint: origin xyz=0 -0.2222 0.37445 rpy=-0.2618 0 0 -> xyz=-0.00015827 -0.22119 0.38344 rpy=-0.2618 0 0
- joint R_shoulder_yaw_joint: origin xyz=0 0.043643 -0.25143 rpy=0.2618 0 0 -> xyz=0 0.043208 -0.25042 rpy=0.2618 0 0
- joint head_yaw_joint: origin xyz=0.012 0 0.617 rpy=0 0 0 -> xyz=0.011342 0 0.62019 rpy=0 0 0

Commit message: 1223_1630_更新了urdf的hip pitch的运动范围，调整了pure cfg

File: general_motion_tracker_whole_body_teleoperation/general_motion_tracker_whole_body_teleoperation/assets/Q1/urdf/Q1_wo_hand_rl.urdf (robot description, URDF)
Before this commit: robot Q1, 30 links, 29 joints
Joints:
- joint L_hip_pitch_joint: limit lower=-0.89 upper=1.64 effort=130 velocity=12.88052988 -> lower=-1.64 upper=0.89 effort=130 velocity=12.88052988
- joint R_hip_pitch_joint: limit lower=-0.89 upper=1.64 effort=130 velocity=12.88052988 -> lower=-1.64 upper=0.89 effort=130 velocity=12.88052988

Commit message: 1231_1654_将电机参数进行了适配

File: general_motion_tracker_whole_body_teleoperation/general_motion_tracker_whole_body_teleoperation/assets/Q1/urdf/Q1_wo_hand_rl.urdf (robot description, URDF)
Before this commit: robot Q1, 30 links, 29 joints
Joints:
- joint L_ankle_pitch_joint: limit lower=-0.87 upper=0.52 effort=0 velocity=0 -> lower=-0.87 upper=0.52 effort=66 velocity=14.660765717
- joint L_ankle_roll_joint: limit lower=-0.26 upper=0.26 effort=0 velocity=0 -> lower=-0.26 upper=0.26 effort=66 velocity=14.660765717
- joint L_elbow_joint: limit lower=-0.87 upper=1.95 effort=0 velocity=0 -> lower=-0.87 upper=1.95 effort=23 velocity=10.157816247
- joint L_forearm_yaw_joint: limit lower=-1.53 upper=1.53 effort=0 velocity=0 -> lower=-1.53 upper=1.53 effort=8.3 velocity=12.356931104
- joint L_hip_pitch_joint: limit lower=-1.64 upper=0.89 effort=0 velocity=0 -> lower=-1.64 upper=0.89 effort=130 velocity=12.88052988
- joint L_hip_roll_joint: limit lower=-0.2 upper=0.83 effort=0 velocity=0 -> lower=-0.2 upper=0.83 effort=72 velocity=14.660765717
- joint L_hip_yaw_joint: limit lower=-0.78 upper=0.78 effort=0 velocity=0 -> lower=-0.78 upper=0.78 effort=55 velocity=12.566370614
- joint L_knee_joint: limit lower=-0.1 upper=2.3 effort=0 velocity=0 -> lower=-0.1 upper=2.3 effort=130 velocity=12.88052988
- joint L_shoulder_pitch_joint: limit lower=-1.48 upper=1.48 effort=0 velocity=0 -> lower=-1.48 upper=1.48 effort=42 velocity=8.58701992
- joint L_shoulder_roll_joint: limit lower=-0.12 upper=3.17 effort=0 velocity=0 -> lower=-0.12 upper=3.17 effort=42 velocity=8.58701992
- joint L_shoulder_yaw_joint: limit lower=-1.69 upper=1.69 effort=0 velocity=0 -> lower=-1.69 upper=1.69 effort=23 velocity=10.157816247
- joint L_wrist_pitch_joint: limit lower=-1.78 upper=1.67 effort=0 velocity=0 -> lower=-1.78 upper=1.67 effort=3.3 velocity=12.356931104
- joint L_wrist_roll_joint: limit lower=-2.3 upper=1.39 effort=0 velocity=0 -> lower=-2.3 upper=1.39 effort=3.3 velocity=12.356931104
- joint R_ankle_pitch_joint: limit lower=-0.87 upper=0.52 effort=0 velocity=0 -> lower=-0.87 upper=0.52 effort=66 velocity=14.660765717
- joint R_ankle_roll_joint: limit lower=-0.26 upper=0.26 effort=0 velocity=0 -> lower=-0.26 upper=0.26 effort=66 velocity=14.660765717
- joint R_elbow_joint: limit lower=-1.95 upper=0.87 effort=0 velocity=0 -> lower=-1.95 upper=0.87 effort=23 velocity=10.157816247
- joint R_forearm_yaw_joint: limit lower=-1.53 upper=1.53 effort=0 velocity=0 -> lower=-1.53 upper=1.53 effort=8.3 velocity=12.356931104
- joint R_hip_pitch_joint: limit lower=-1.64 upper=0.89 effort=0 velocity=0 -> lower=-1.64 upper=0.89 effort=130 velocity=12.88052988
- joint R_hip_roll_joint: limit lower=-0.83 upper=0.2 effort=0 velocity=0 -> lower=-0.83 upper=0.2 effort=72 velocity=14.660765717
- joint R_hip_yaw_joint: limit lower=-0.78 upper=0.78 effort=0 velocity=0 -> lower=-0.78 upper=0.78 effort=55 velocity=12.566370614
- joint R_knee_joint: limit lower=-0.1 upper=2.3 effort=0 velocity=0 -> lower=-0.1 upper=2.3 effort=130 velocity=12.88052988
- joint R_shoulder_pitch_joint: limit lower=-1.48 upper=1.48 effort=0 velocity=0 -> lower=-1.48 upper=1.48 effort=42 velocity=8.58701992
- joint R_shoulder_roll_joint: limit lower=-3.17 upper=0.12 effort=0 velocity=0 -> lower=-3.17 upper=0.12 effort=42 velocity=8.58701992
- joint R_shoulder_yaw_joint: limit lower=-1.69 upper=1.69 effort=0 velocity=0 -> lower=-1.69 upper=1.69 effort=23 velocity=10.157816247
- joint R_wrist_pitch_joint: limit lower=-1.78 upper=1.67 effort=0 velocity=0 -> lower=-1.78 upper=1.67 effort=3.3 velocity=12.356931104
- joint R_wrist_roll_joint: limit lower=-1.39 upper=2.3 effort=0 velocity=0 -> lower=-1.39 upper=2.3 effort=3.3 velocity=12.356931104
- joint head_pitch_joint: limit lower=-0.38 upper=0.33 effort=0 velocity=0 -> lower=-0.38 upper=0.33 effort=1.26 velocity=58.433623357
- joint head_yaw_joint: limit lower=-1.57 upper=1.57 effort=0 velocity=0 -> lower=-1.57 upper=1.57 effort=2.52 velocity=29.216811679
- joint pelvis_joint: limit lower=-1.04 upper=1.04 effort=0 velocity=0 -> lower=-1.04 upper=1.04 effort=42 velocity=8.58701992

Commit message: 0106_1915_修正了URDF中pelvis_link的质量、惯量属性

File: general_motion_tracker_whole_body_teleoperation/general_motion_tracker_whole_body_teleoperation/assets/Q1/urdf/Q1_wo_hand_rl.urdf (robot description, URDF)
Before this commit: robot Q1, 30 links, 29 joints
Links:
- link pelvis_link: mass 4.9667 -> 6.0067291
