Commit message: 1231_1401_新版Q1的URDF更新

File: general_motion_tracker_whole_body_teleoperation/general_motion_tracker_whole_body_teleoperation/assets/Q1/urdf/Q1.urdf (robot description, URDF)
Before this commit: robot Q1, 30 links, 29 joints
Links:
- added link world
- link L_ankle_pitch_link: geometry collision cylinder length=0.001 radius=0.001; visual mesh filename=package://Q1/meshes/L_ankle_pitch_link.STL
- link L_ankle_roll_link: geometry collision sphere radius=0.005; collision sphere radius=0.005
- link L_elbow_link: geometry collision cylinder length=0.03 radius=0.02; visual mesh filename=package://Q1/meshes/L_elbow_link.STL
- link L_forearm_yaw_link: geometry collision cylinder length=0.03 radius=0.025; visual mesh filename=package://Q1/meshes/L_forearm_yaw_link.STL
- link L_hip_pitch_link: geometry collision cylinder length=0.09 radius=0.025; visual mesh filename=package://Q1/meshes/L_hip_pitch_link.STL
- link L_hip_roll_link: geometry collision cylinder length=0.017 radius=0.025; visual mesh filename=package://Q1/meshes/L_hip_roll_link.STL
- link L_hip_yaw_link: geometry collision cylinder length=0.04 radius=0.025; visual mesh filename=package://Q1/meshes/L_hip_yaw_link.STL
- link L_knee_link: geometry collision cylinder length=0.1 radius=0.025; collision cylinder length=0.1 radius=0.025
- link L_shoulder_pitch_link: geometry collision cylinder length=0.03 radius=0.025; visual mesh filename=package://Q1/meshes/L_shoulder_pitch_link.STL
- link L_shoulder_roll_link: geometry collision cylinder length=0.03 radius=0.02; visual mesh filename=package://Q1/meshes/L_shoulder_roll_link.STL
- link L_shoulder_yaw_link: geometry collision cylinder length=0.06 radius=0.02; visual mesh filename=package://Q1/meshes/L_shoulder_yaw_link.STL
- link L_wrist_pitch_link: geometry collision box size=0.06 0.03 0.18; visual mesh filename=package://Q1/meshes/L_wrist_pitch_link.STL
- link L_wrist_roll_link: geometry collision cylinder length=0.01 radius=0.015; visual mesh filename=package://Q1/meshes/L_wrist_roll_link.STL
- link R_ankle_pitch_link: geometry collision cylinder length=0.001 radius=0.001; visual mesh filename=package://Q1/meshes/R_ankle_pitch_link.STL
- link R_ankle_roll_link: geometry collision sphere radius=0.005; collision sphere radius=0.005
- link R_elbow_link: geometry collision cylinder length=0.03 radius=0.02; visual mesh filename=package://Q1/meshes/R_elbow_link.STL
- link R_forearm_yaw_link: geometry collision cylinder length=0.03 radius=0.025; visual mesh filename=package://Q1/meshes/R_forearm_yaw_link.STL
- link R_hip_pitch_link: geometry collision cylinder length=0.09 radius=0.025; visual mesh filename=package://Q1/meshes/R_hip_pitch_link.STL
- link R_hip_roll_link: geometry collision cylinder length=0.017 radius=0.025; visual mesh filename=package://Q1/meshes/R_hip_roll_link.STL
- link R_hip_yaw_link: geometry collision cylinder length=0.04 radius=0.025; visual mesh filename=package://Q1/meshes/R_hip_yaw_link.STL
- link R_knee_link: geometry collision cylinder length=0.1 radius=0.025; collision cylinder length=0.1 radius=0.025
- link R_shoulder_pitch_link: geometry collision cylinder length=0.03 radius=0.025; visual mesh filename=package://Q1/meshes/R_shoulder_pitch_link.STL
- link R_shoulder_roll_link: geometry collision cylinder length=0.03 radius=0.02; visual mesh filename=package://Q1/meshes/R_shoulder_roll_link.STL
- link R_shoulder_yaw_link: geometry collision cylinder length=0.06 radius=0.02; visual mesh filename=package://Q1/meshes/R_shoulder_yaw_link.STL
- link R_wrist_pitch_link: geometry collision box size=0.06 0.03 0.18; visual mesh filename=package://Q1/meshes/R_wrist_pitch_link.STL
- link R_wrist_roll_link: geometry collision cylinder length=0.01 radius=0.015; visual mesh filename=package://Q1/meshes/R_wrist_roll_link.STL
- link head_pitch_link: geometry collision box size=0.01 0.12 0.12; visual mesh filename=package://Q1/meshes/head_pitch_link.STL
- link head_yaw_link: geometry collision box size=0.01 0.01 0.01; visual mesh filename=package://Q1/meshes/head_yaw_link.STL
- link pelvis_link: geometry collision box size=0.08 0.35 0.1; visual mesh filename=package://Q1/meshes/pelvis_link.STL
- link torso_link: geometry collision box size=0.25 0.16 0.37; visual mesh filename=package://Q1/meshes/torso_link.STL
Joints:
- added joint floating_base_joint: type floating, parent world, child pelvis_link

Commit message: update Q1 urdf

File: general_motion_tracker_whole_body_teleoperation/general_motion_tracker_whole_body_teleoperation/assets/Q1/urdf/Q1.urdf (robot description, URDF)
Before this commit: robot Q1, 31 links, 30 joints
Links:
- removed link L_forearm_yaw_link
- removed link R_forearm_yaw_link
- removed link world
- added link L_wrist_yaw_link, mass 0.16; collision mesh filename=package://Q1/meshes/L_wrist_yaw_link.STL; visual mesh filename=package://Q1/meshes/L_wrist_yaw_link.STL
- added link R_wrist_yaw_link, mass 0.16; collision mesh filename=package://Q1/meshes/R_wrist_yaw_link.STL; visual mesh filename=package://Q1/meshes/R_wrist_yaw_link.STL
- link L_ankle_pitch_link: mass 0.046144 -> 0.046; geometry collision mesh filename=package://Q1/meshes/L_ankle_pitch_link.STL; visual mesh filename=package://Q1/meshes/L_ankle_pitch_link.STL
- link L_ankle_roll_link: geometry collision mesh filename=package://Q1/meshes/L_ankle_roll_link.STL; visual mesh filename=package://Q1/meshes/L_ankle_roll_link.STL
- link L_elbow_link: geometry collision mesh filename=package://Q1/meshes/L_elbow_link.STL; visual mesh filename=package://Q1/meshes/L_elbow_link.STL
- link L_hip_pitch_link: mass 2.0912 -> 2.0912352; geometry collision mesh filename=package://Q1/meshes/L_hip_pitch_link.STL; visual mesh filename=package://Q1/meshes/L_hip_pitch_link.STL
- link L_hip_roll_link: mass 1.4404 -> 1.6267; geometry collision mesh filename=package://Q1/meshes/L_hip_roll_link.STL; visual mesh filename=package://Q1/meshes/L_hip_roll_link.STL
- link L_hip_yaw_link: mass 3.6555 -> 3.6555048; geometry collision mesh filename=package://Q1/meshes/L_hip_yaw_link.STL; visual mesh filename=package://Q1/meshes/L_hip_yaw_link.STL
- link L_knee_link: mass 7.5002 -> 7.5002071; geometry collision mesh filename=package://Q1/meshes/L_knee_link.STL; visual mesh filename=package://Q1/meshes/L_knee_link.STL
- link L_shoulder_pitch_link: geometry collision mesh filename=package://Q1/meshes/L_shoulder_pitch_link.STL; visual mesh filename=package://Q1/meshes/L_shoulder_pitch_link.STL
- link L_shoulder_roll_link: geometry collision mesh filename=package://Q1/meshes/L_shoulder_roll_link.STL; visual mesh filename=package://Q1/meshes/L_shoulder_roll_link.STL
- link L_shoulder_yaw_link: geometry collision mesh filename=package://Q1/meshes/L_shoulder_yaw_link.STL; visual mesh filename=package://Q1/meshes/L_shoulder_yaw_link.STL
- link L_wrist_pitch_link: mass 0.16 -> 0.25; geometry collision mesh filename=package://Q1/meshes/L_wrist_pitch_link.STL; visual mesh filename=package://Q1/meshes/L_wrist_pitch_link.STL
- link L_wrist_roll_link: mass 0.25 -> 1.05; geometry collision mesh filename=package://Q1/meshes/L_wrist_roll_link.STL; visual mesh filename=package://Q1/meshes/L_wrist_roll_link.STL
- link R_ankle_pitch_link: geometry collision mesh filename=package://Q1/meshes/R_ankle_pitch_link.STL; visual mesh filename=package://Q1/meshes/R_ankle_pitch_link.STL
- link R_ankle_roll_link: geometry collision mesh filename=package://Q1/meshes/R_ankle_roll_link.STL; visual mesh filename=package://Q1/meshes/R_ankle_roll_link.STL
- link R_elbow_link: geometry collision mesh filename=package://Q1/meshes/R_elbow_link.STL; visual mesh filename=package://Q1/meshes/R_elbow_link.STL
- link R_hip_pitch_link: mass 2.0922 -> 2.0922344; geometry collision mesh filename=package://Q1/meshes/R_hip_pitch_link.STL; visual mesh filename=package://Q1/meshes/R_hip_pitch_link.STL
- link R_hip_roll_link: mass 1.4404 -> 1.6267; geometry collision mesh filename=package://Q1/meshes/R_hip_roll_link.STL; visual mesh filename=package://Q1/meshes/R_hip_roll_link.STL
- link R_hip_yaw_link: mass 3.6555 -> 3.6554644; geometry collision mesh filename=package://Q1/meshes/R_hip_yaw_link.STL; visual mesh filename=package://Q1/meshes/R_hip_yaw_link.STL
- link R_knee_link: mass 7.5025 -> 7.502175; geometry collision mesh filename=package://Q1/meshes/R_knee_link.STL; visual mesh filename=package://Q1/meshes/R_knee_link.STL
- link R_shoulder_pitch_link: geometry collision mesh filename=package://Q1/meshes/R_shoulder_pitch_link.STL; visual mesh filename=package://Q1/meshes/R_shoulder_pitch_link.STL
- link R_shoulder_roll_link: geometry collision mesh filename=package://Q1/meshes/R_shoulder_roll_link.STL; visual mesh filename=package://Q1/meshes/R_shoulder_roll_link.STL
- link R_shoulder_yaw_link: geometry collision mesh filename=package://Q1/meshes/R_shoulder_yaw_link.STL; visual mesh filename=package://Q1/meshes/R_shoulder_yaw_link.STL
- link R_wrist_pitch_link: mass 0.16 -> 0.25; geometry collision mesh filename=package://Q1/meshes/R_wrist_pitch_link.STL; visual mesh filename=package://Q1/meshes/R_wrist_pitch_link.STL
- link R_wrist_roll_link: mass 0.25 -> 1.05; geometry collision mesh filename=package://Q1/meshes/R_wrist_roll_link.STL; visual mesh filename=package://Q1/meshes/R_wrist_roll_link.STL
- link head_pitch_link: geometry collision mesh filename=package://Q1/meshes/head_pitch_link.STL; visual mesh filename=package://Q1/meshes/head_pitch_link.STL
- link head_yaw_link: geometry collision mesh filename=package://Q1/meshes/head_yaw_link.STL; visual mesh filename=package://Q1/meshes/head_yaw_link.STL
- link pelvis_link: mass 4.9667 -> 8.1798; geometry collision mesh filename=package://Q1/meshes/pelvis_link.STL; visual mesh filename=package://Q1/meshes/pelvis_link.STL
- link torso_link: mass 17.278 -> 19.21; geometry collision mesh filename=package://Q1/meshes/torso_link.STL; visual mesh filename=package://Q1/meshes/torso_link.STL
Joints:
- removed joint L_forearm_yaw_joint
- removed joint R_forearm_yaw_joint
- removed joint floating_base_joint
- added joint L_wrist_yaw_joint: type revolute, parent L_wrist_pitch_link, child L_wrist_yaw_link, origin xyz=0 0 0 rpy=0 0 0, axis 0 1 0, limit lower=-1.78 upper=1.67 effort=8.3 velocity=12.35
- added joint R_wrist_yaw_joint: type revolute, parent R_wrist_pitch_link, child R_wrist_yaw_link, origin xyz=0 0 0 rpy=0 0 0, axis 0 1 0, limit lower=-1.78 upper=1.67 effort=8.3 velocity=12.35
- joint L_ankle_pitch_joint: limit lower=-0.87 upper=0.52 effort=0 velocity=0 -> lower=-0.52 upper=0.87 effort=66 velocity=14.66
- joint L_ankle_roll_joint: limit lower=-0.26 upper=0.26 effort=0 velocity=0 -> lower=-0.4363 upper=0.4363 effort=66 velocity=14.66
- joint L_elbow_joint: axis 0 1 0 -> 1 0 0; limit lower=-0.87 upper=1.95 effort=0 velocity=0 -> lower=-1.95 upper=0.87 effort=23 velocity=10.15
- joint L_hip_pitch_joint: limit lower=-1.64 upper=0.89 effort=0 velocity=0 -> lower=-0.89 upper=1.64 effort=130 velocity=12.88
- joint L_hip_roll_joint: limit lower=-0.2 upper=0.83 effort=0 velocity=0 -> lower=-0.2 upper=0.83 effort=130 velocity=12.88; origin xyz=-0.00010006 0.125 -0.059738 rpy=0 0 0 -> xyz=0.0154 0.125 -0.062997 rpy=0 0 0
- joint L_hip_yaw_joint: limit lower=-0.78 upper=0.78 effort=0 velocity=0 -> lower=-0.78 upper=0.78 effort=55 velocity=12.56
- joint L_knee_joint: limit lower=-0.1 upper=2.3 effort=0 velocity=0 -> lower=-0.1 upper=2.3 effort=130 velocity=12.88
- joint L_shoulder_pitch_joint: limit lower=-1.48 upper=1.48 effort=0 velocity=0 -> lower=-1.48 upper=1.48 effort=42 velocity=8.58; origin xyz=-0.00015827 0.22119 0.38344 rpy=0.2618 0 0 -> xyz=0.015442 0.22168 0.37829 rpy=0.2618 0 0
- joint L_shoulder_roll_joint: limit lower=-0.12 upper=3.17 effort=0 velocity=0 -> lower=-0.12 upper=3.17 effort=42 velocity=8.58
- joint L_shoulder_yaw_joint: limit lower=-1.69 upper=1.69 effort=0 velocity=0 -> lower=-1.69 upper=1.69 effort=23 velocity=10.15; origin xyz=0 -0.043208 -0.25042 rpy=-0.2618 0 0 -> xyz=0 -0.043708 -0.2504 rpy=-0.2618 0 0
- joint L_wrist_pitch_joint: axis 0 1 0 -> 1 0 0; limit lower=-1.78 upper=1.67 effort=0 velocity=0 -> lower=-2.3 upper=1.39 effort=8.3 velocity=12.35
- joint L_wrist_roll_joint: axis 1 0 0 -> 0 0 1; limit lower=-2.3 upper=1.39 effort=0 velocity=0 -> lower=-1.53 upper=1.53 effort=8.3 velocity=12.35; origin xyz=0 0 0 rpy=0 0 0 -> xyz=0 0 -0.211 rpy=0 0 0; parent L_forearm_yaw_link -> L_elbow_link
- joint R_ankle_pitch_joint: limit lower=-0.87 upper=0.52 effort=0 velocity=0 -> lower=-0.52 upper=0.87 effort=66 velocity=14.66
- joint R_ankle_roll_joint: limit lower=-0.26 upper=0.26 effort=0 velocity=0 -> lower=-0.4363 upper=0.4363 effort=66 velocity=14.66
- joint R_elbow_joint: axis 0 1 0 -> 1 0 0; limit lower=-1.95 upper=0.87 effort=0 velocity=0 -> lower=-0.87 upper=1.95 effort=23 velocity=10.15
- joint R_hip_pitch_joint: limit lower=-1.64 upper=0.89 effort=0 velocity=0 -> lower=-0.89 upper=1.64 effort=130 velocity=12.88
- joint R_hip_roll_joint: limit lower=-0.83 upper=0.2 effort=0 velocity=0 -> lower=-0.83 upper=0.2 effort=130 velocity=12.88; origin xyz=-0.00010006 -0.125 -0.059738 rpy=0 0 0 -> xyz=0.0154 -0.125 -0.062997 rpy=0 0 0
- joint R_hip_yaw_joint: limit lower=-0.78 upper=0.78 effort=0 velocity=0 -> lower=-0.78 upper=0.78 effort=55 velocity=12.56
- joint R_knee_joint: limit lower=-0.1 upper=2.3 effort=0 velocity=0 -> lower=-0.1 upper=2.3 effort=130 velocity=12.88
- joint R_shoulder_pitch_joint: limit lower=-1.48 upper=1.48 effort=0 velocity=0 -> lower=-1.48 upper=1.48 effort=42 velocity=8.58; origin xyz=-0.00015827 -0.22119 0.38344 rpy=-0.2618 0 0 -> xyz=0.015442 -0.22168 0.37829 rpy=-0.2618 0 0
- joint R_shoulder_roll_joint: limit lower=-3.17 upper=0.12 effort=0 velocity=0 -> lower=-3.17 upper=0.12 effort=42 velocity=8.58
- joint R_shoulder_yaw_joint: limit lower=-1.69 upper=1.69 effort=0 velocity=0 -> lower=-1.69 upper=1.69 effort=23 velocity=10.15; origin xyz=0 0.043208 -0.25042 rpy=0.2618 0 0 -> xyz=0 0.043708 -0.2504 rpy=0.2618 0 0
- joint R_wrist_pitch_joint: axis 0 1 0 -> 1 0 0; limit lower=-1.78 upper=1.67 effort=0 velocity=0 -> lower=-1.39 upper=2.3 effort=8.3 velocity=12.35
- joint R_wrist_roll_joint: axis 1 0 0 -> 0 0 1; limit lower=-1.39 upper=2.3 effort=0 velocity=0 -> lower=-1.53 upper=1.53 effort=8.3 velocity=12.35; origin xyz=0 0 0 rpy=0 0 0 -> xyz=0 0 -0.211 rpy=0 0 0; parent R_forearm_yaw_link -> R_elbow_link
- joint head_pitch_joint: limit lower=-0.38 upper=0.33 effort=0 velocity=0 -> lower=-0.38 upper=0.33 effort=2.52 velocity=29.21
- joint head_yaw_joint: limit lower=-1.57 upper=1.57 effort=0 velocity=0 -> lower=-1.57 upper=1.57 effort=2.52 velocity=29.21; origin xyz=0.011342 0 0.62019 rpy=0 0 0 -> xyz=0.026942 0 0.61493 rpy=0 0 0
- joint pelvis_joint: child torso_link -> pelvis_link; limit lower=-1.04 upper=1.04 effort=0 velocity=0 -> lower=-1.04 upper=1.04 effort=130 velocity=12.88; parent pelvis_link -> torso_link

File: general_motion_tracker_whole_body_teleoperation/general_motion_tracker_whole_body_teleoperation/assets/Q1/urdf/Q1_wo_hand_rl.urdf (robot description, URDF)
Before this commit: robot Q1, 30 links, 29 joints
Links:
- link L_ankle_pitch_link: mass 0.046144 -> 0.046
- link L_hip_pitch_link: mass 2.0912 -> 2.0912352
- link L_hip_roll_link: mass 1.4404 -> 1.6267
- link L_hip_yaw_link: mass 3.6555 -> 3.6555048
- link L_knee_link: mass 7.5002 -> 7.5002071
- link R_hip_pitch_link: mass 2.0922 -> 2.0922344
- link R_hip_roll_link: mass 1.4404 -> 1.6267
- link R_hip_yaw_link: mass 3.6555 -> 3.6554644
- link R_knee_link: mass 7.5025 -> 7.502175
- link head_pitch_link: geometry collision mesh filename=meshes/head_pitch_link.STL; visual mesh filename=meshes/head_pitch_link.STL
- link head_yaw_link: geometry collision mesh filename=meshes/head_yaw_link.STL; visual mesh filename=meshes/head_yaw_link.STL
- link pelvis_link: mass 6.0067291 -> 8.1798
- link torso_link: mass 17.278 -> 19.21
Joints:
- joint L_ankle_pitch_joint: limit lower=-0.87 upper=0.52 effort=66 velocity=14.660765717 -> lower=-0.52 upper=0.87 effort=66 velocity=14.66
- joint L_ankle_roll_joint: limit lower=-0.26 upper=0.26 effort=66 velocity=14.660765717 -> lower=-0.4363 upper=0.4363 effort=66 velocity=14.66
- joint L_elbow_joint: limit lower=-0.87 upper=1.95 effort=23 velocity=10.157816247 -> lower=-1.95 upper=0.87 effort=23 velocity=10.15
- joint L_forearm_yaw_joint: limit lower=-1.53 upper=1.53 effort=8.3 velocity=12.356931104 -> lower=-1.53 upper=1.53 effort=8.3 velocity=12.35; origin xyz=0 0 -0.209 rpy=0 0 0 -> xyz=0 0 -0.211 rpy=0 0 0
- joint L_hip_pitch_joint: limit lower=-1.64 upper=0.89 effort=130 velocity=12.88052988 -> lower=-0.89 upper=1.64 effort=130 velocity=12.88
- joint L_hip_roll_joint: limit lower=-0.2 upper=0.83 effort=72 velocity=14.660765717 -> lower=-0.2 upper=0.83 effort=130 velocity=12.88; origin xyz=-0.00010006 0.125 -0.059738 rpy=0 0 0 -> xyz=0.0154 0.125 -0.062997 rpy=0 0 0
- joint L_hip_yaw_joint: limit lower=-0.78 upper=0.78 effort=55 velocity=12.566370614 -> lower=-0.78 upper=0.78 effort=55 velocity=12.56
- joint L_knee_joint: limit lower=-0.1 upper=2.3 effort=130 velocity=12.88052988 -> lower=-0.1 upper=2.3 effort=130 velocity=12.88
- joint L_shoulder_pitch_joint: limit lower=-1.48 upper=1.48 effort=42 velocity=8.58701992 -> lower=-1.48 upper=1.48 effort=42 velocity=8.58; origin xyz=-0.00015827 0.22119 0.38344 rpy=0.2618 0 0 -> xyz=0.015442 0.22168 0.37829 rpy=0.2618 0 0
- joint L_shoulder_roll_joint: limit lower=-0.12 upper=3.17 effort=42 velocity=8.58701992 -> lower=-0.12 upper=3.17 effort=42 velocity=8.58
- joint L_shoulder_yaw_joint: limit lower=-1.69 upper=1.69 effort=23 velocity=10.157816247 -> lower=-1.69 upper=1.69 effort=23 velocity=10.15; origin xyz=0 -0.043208 -0.25042 rpy=-0.2618 0 0 -> xyz=0 -0.043708 -0.2504 rpy=-0.2618 0 0
- joint L_wrist_pitch_joint: limit lower=-1.78 upper=1.67 effort=3.3 velocity=12.356931104 -> lower=-1.78 upper=1.67 effort=8.3 velocity=12.35
- joint L_wrist_roll_joint: limit lower=-2.3 upper=1.39 effort=3.3 velocity=12.356931104 -> lower=-2.3 upper=1.39 effort=8.3 velocity=12.35
- joint R_ankle_pitch_joint: limit lower=-0.87 upper=0.52 effort=66 velocity=14.660765717 -> lower=-0.52 upper=0.87 effort=66 velocity=14.66
- joint R_ankle_roll_joint: limit lower=-0.26 upper=0.26 effort=66 velocity=14.660765717 -> lower=-0.4363 upper=0.4363 effort=66 velocity=14.66
- joint R_elbow_joint: limit lower=-1.95 upper=0.87 effort=23 velocity=10.157816247 -> lower=-0.87 upper=1.95 effort=23 velocity=10.15
- joint R_forearm_yaw_joint: limit lower=-1.53 upper=1.53 effort=8.3 velocity=12.356931104 -> lower=-1.53 upper=1.53 effort=8.3 velocity=12.35; origin xyz=0 0 -0.209 rpy=0 0 0 -> xyz=0 0 -0.211 rpy=0 0 0
- joint R_hip_pitch_joint: limit lower=-1.64 upper=0.89 effort=130 velocity=12.88052988 -> lower=-0.89 upper=1.64 effort=130 velocity=12.88
- joint R_hip_roll_joint: limit lower=-0.83 upper=0.2 effort=72 velocity=14.660765717 -> lower=-0.83 upper=0.2 effort=130 velocity=12.88; origin xyz=-0.00010006 -0.125 -0.059738 rpy=0 0 0 -> xyz=0.0154 -0.125 -0.062997 rpy=0 0 0
- joint R_hip_yaw_joint: limit lower=-0.78 upper=0.78 effort=55 velocity=12.566370614 -> lower=-0.78 upper=0.78 effort=55 velocity=12.56
- joint R_knee_joint: limit lower=-0.1 upper=2.3 effort=130 velocity=12.88052988 -> lower=-0.1 upper=2.3 effort=130 velocity=12.88
- joint R_shoulder_pitch_joint: limit lower=-1.48 upper=1.48 effort=42 velocity=8.58701992 -> lower=-1.48 upper=1.48 effort=42 velocity=8.58; origin xyz=-0.00015827 -0.22119 0.38344 rpy=-0.2618 0 0 -> xyz=0.015442 -0.22168 0.37829 rpy=-0.2618 0 0
- joint R_shoulder_roll_joint: limit lower=-3.17 upper=0.12 effort=42 velocity=8.58701992 -> lower=-3.17 upper=0.12 effort=42 velocity=8.58
- joint R_shoulder_yaw_joint: limit lower=-1.69 upper=1.69 effort=23 velocity=10.157816247 -> lower=-1.69 upper=1.69 effort=23 velocity=10.15; origin xyz=0 0.043208 -0.25042 rpy=0.2618 0 0 -> xyz=0 0.043708 -0.2504 rpy=0.2618 0 0
- joint R_wrist_pitch_joint: limit lower=-1.78 upper=1.67 effort=3.3 velocity=12.356931104 -> lower=-1.78 upper=1.67 effort=8.3 velocity=12.35
- joint R_wrist_roll_joint: limit lower=-1.39 upper=2.3 effort=3.3 velocity=12.356931104 -> lower=-1.39 upper=2.3 effort=8.3 velocity=12.35
- joint head_pitch_joint: limit lower=-0.38 upper=0.33 effort=1.26 velocity=58.433623357 -> lower=-0.38 upper=0.33 effort=2.52 velocity=29.21
- joint head_yaw_joint: limit lower=-1.57 upper=1.57 effort=2.52 velocity=29.216811679 -> lower=-1.57 upper=1.57 effort=2.52 velocity=29.21; origin xyz=0.011342 0 0.62019 rpy=0 0 0 -> xyz=0.026942 0 0.61493 rpy=0 0 0
- joint pelvis_joint: limit lower=-1.04 upper=1.04 effort=42 velocity=8.58701992 -> lower=-1.04 upper=1.04 effort=130 velocity=12.88
